Commit message: udpated max and min robot arm movement

File: ros_ws/src/xarm_description/urdf/xarm.urdf (robot description, URDF)
Before this commit: robot xarm, 5 links, 5 joints
Joints:
- joint xarm_2_joint: limit lower=-1.208 upper=1.933 effort=1000 velocity=1.0 -> lower=-2.35 upper=2.35 effort=1000 velocity=1.0
- joint xarm_3_joint: limit lower=-1.740612146 upper=1.86797401 effort=1000 velocity=1.0 -> lower=-2.05 upper=2.35 effort=1000 velocity=1.0
- joint xarm_4_joint: limit lower=-1.910427965 upper=1.910427965 effort=1000 velocity=1.0 -> lower=-2.2 upper=2.2 effort=1000 velocity=1.0
- joint xarm_5_joint: limit lower=-1.592023304 upper=1.86797401 effort=1000 velocity=1.0 -> lower=-1.62 upper=1.62 effort=1000 velocity=1.0
- joint xarm_6_joint: limit lower=-1.737238322 upper=1.79965407 effort=1000 velocity=1.0 -> lower=-2.35 upper=2.35 effort=1000 velocity=1.0

File: ros_ws/src/xarm_description/urdf/xarm_v2.urdf (robot description, URDF)
Before this commit: robot xarm, 5 links, 5 joints
Joints:
- joint xarm_2_joint: limit lower=-1.208 upper=1.933 effort=1000 velocity=1.0 -> lower=-2.35 upper=2.35 effort=1000 velocity=1.0
- joint xarm_3_joint: limit lower=-1.740612146 upper=1.86797401 effort=1000 velocity=1.0 -> lower=-2.05 upper=2.35 effort=1000 velocity=1.0
- joint xarm_4_joint: limit lower=-1.910427965 upper=1.910427965 effort=1000 velocity=1.0 -> lower=-2.2 upper=2.2 effort=1000 velocity=1.0
- joint xarm_5_joint: limit lower=-1.592023304 upper=1.86797401 effort=1000 velocity=1.0 -> lower=-1.62 upper=1.62 effort=1000 velocity=1.0
- joint xarm_6_joint: limit lower=-1.737238322 upper=1.79965407 effort=1000 velocity=1.0 -> lower=-2.35 upper=2.35 effort=1000 velocity=1.0
