Commit message: gripper stuff

File: ros_ws/src/xarm_description/urdf/ros2_control.arm.xacro (robot description, xacro)
@@ -28,10 +28,8 @@
         </joint>
         <!-- mirror here -->
-       <!-- <joint name="xarm_1_joint_mirror">
-            <param name="mimic">xarm_1_joint</param>
-            <param name="multiplier">-1</param>
-            <state_interface name="position"/>
-            <state_interface name="velocity"/>
-        </joint> -->
+       <joint name="xarm_1_joint_mirror">
+            <state_interface name="position"/>
+            <state_interface name="velocity"/>
+        </joint>
       </xacro:if>
       <xacro:if value="${eef == 'eef_3_finger'}">
@@ -131,6 +129,6 @@
                 <multiplier>-1</multiplier>
             </param> -->
-            <param name="mimic">xarm_1_joint</param>
-            <param name="multiplier">-1</param>
+            <!-- <param name="mimic">xarm_1_joint</param>
+            <param name="multiplier">-1</param> -->
             <state_interface name="position"/>
             <state_interface name="velocity"/>

Commit message: mirror reversed

File: ros_ws/src/xarm_description/urdf/ros2_control.arm.xacro (robot description, xacro)
@@ -28,8 +28,8 @@
         </joint>
         <!-- mirror here -->
-       <joint name="xarm_1_joint_mirror">
-            <state_interface name="position"/>
-            <state_interface name="velocity"/>
-        </joint>
+       <!-- <joint name="xarm_1_joint_mirror">
+            <state_interface name="position"/>
+            <state_interface name="velocity"/>
+        </joint> -->
       </xacro:if>
       <xacro:if value="${eef == 'eef_3_finger'}">

Commit message: mirror fixed

File: ros_ws/src/xarm_description/urdf/ros2_control.arm.xacro (robot description, xacro)
@@ -28,8 +28,8 @@
         </joint>
         <!-- mirror here -->
-       <!-- <joint name="xarm_1_joint_mirror">
-            <state_interface name="position"/>
-            <state_interface name="velocity"/>
-        </joint> -->
+       <joint name="xarm_1_joint_mirror">
+            <state_interface name="position"/>
+            <state_interface name="velocity"/>
+        </joint>
       </xacro:if>
       <xacro:if value="${eef == 'eef_3_finger'}">
