Commit message: updates

File: ros_ws/src/xarm_description/urdf/xarm_v2.urdf (robot description, URDF)
Before this commit: robot xarm, 5 links, 5 joints
Joints:
- joint xarm_3_joint: axis 1 0 0 -> -1 0 0
- joint xarm_5_joint: axis 1 0 0 -> -1 0 0

Commit message: updates

File: ros_ws/src/xarm_description/urdf/xarm_v2.urdf (robot description, URDF)
Before this commit: robot xarm, 5 links, 5 joints
Links:
- added link eef_2_finger_left_link, mass 0.1; collision mesh filename=file://$(find xarm_description)/meshes/stls/gripper_finger_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 scale=1.0 1.0 1.0; visual mesh filename=file://$(find xarm_description)/meshes/stls/gripper_finger_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 scale=1.0 1.0 1.0
- added link eef_2_finger_right_link, mass 0.1; collision mesh filename=file://$(find xarm_description)/meshes/stls/gripper_finger_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 scale=1.0 1.0 1.0; visual mesh filename=file://$(find xarm_description)/meshes/stls/gripper_finger_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 scale=1.0 1.0 1.0
- added link eef_base_link, mass 0.1; collision mesh filename=file://$(find xarm_description)/meshes/stls/gripper_palm.stl scale=1.0 1.0 1.0; visual mesh filename=file://$(find xarm_description)/meshes/stls/gripper_palm.stl scale=1.0 1.0 1.0
Joints:
- added joint xarm_1_joint: type prismatic, parent eef_base_link, child eef_2_finger_left_link, origin xyz=0 0 0.050 rpy=0 0 0, axis 1 0 0, limit lower=0.00 upper=0.028 effort=1000.0 velocity=0.5
- added joint xarm_1_joint_mirror: type prismatic, parent eef_base_link, child eef_2_finger_right_link, origin xyz=0 0 0.050 rpy=0 0 0, axis 1 0 0, limit lower=0.003 upper=0.028 effort=1000.0 velocity=0.5, mimic joint=xarm_1_joint multiplier=-1.0
- joint xarm_2_joint: child (none) -> eef_base_link

Commit message: got ik working

File: ros_ws/src/xarm_description/urdf/xarm_v2.urdf (robot description, URDF)
Before this commit: robot xarm, 8 links, 7 joints
Joints:
- joint xarm_3_joint: axis -1 0 0 -> 1 0 0
- joint xarm_4_joint: axis 1 0 0 -> -1 0 0
- joint xarm_5_joint: axis -1 0 0 -> 1 0 0

Commit message: finger pinch

File: ros_ws/src/xarm_description/urdf/xarm_v2.urdf (robot description, URDF)
Before this commit: robot xarm, 8 links, 7 joints
Links:
- added link finger_pinch_link
Joints:
- added joint finger_pinch_joint: type fixed, parent eef_base_link, child finger_pinch_link, origin xyz=0 0 0.09 rpy=0 0 0

Commit message: update length

File: ros_ws/src/xarm_description/urdf/xarm_v2.urdf (robot description, URDF)
Before this commit: robot xarm, 9 links, 8 joints
Joints:
- joint xarm_3_joint: origin xyz=0 0.0 0.093 rpy=0 0 0 -> xyz=0 0.0 0.095 rpy=0 0 0

Commit message: image sync to improve distance

File: ros_ws/src/xarm_description/urdf/xarm_v2.urdf (robot description, URDF)
Before this commit: robot xarm, 9 links, 8 joints
Joints:
- joint finger_pinch_joint: origin xyz=0 0 0.09 rpy=0 0 0 -> xyz=0 0 0.11 rpy=0 0 0
