Commit message: update camera pan tilt

File: ros_ws/src/autonomous_robot/description/pan_tilt_xacros/pan_tilt.xacro (robot description, xacro)
@@ -17,6 +17,12 @@
     <xacro:property name="camera_width" value="0.025"/>
     <xacro:property name="camera_height" value="0.025"/>
+    <xacro:property name="camera_mount_l" value="0.09"/>
+    <xacro:property name="camera_mount_w" value="0.068"/>
+    <xacro:property name="camera_mount_h" value="0.085"/>
+    <xacro:property name="pan_tilt_leg_l" value="0.025"/>
+    <xacro:property name="pan_tilt_leg_2" value="0.058"/>
+    <xacro:property name="pan_tilt_leg_h" value="0.065"/>
     <!-- Mount Properties -->
-    <xacro:property name="mount_thickness" value="0.003"/>
+    <xacro:property name="mount_thickness" value="0.0052"/>
     <xacro:property name="bracket_height" value="0.04"/>
     <!-- Materials -->
@@ -122,18 +128,20 @@
     <link name="pan_link">
       <visual>
+        <origin xyz="0 0 0" rpy="0 0 0"/>
+        <geometry>
+          <mesh filename="file://$(find image_sync_processor)/meshes/stls/PAN-TILT_ROTOR_V2_fixed.stl" scale="0.001 0.001 0.001" />
+          <!-- <box size="${mount_thickness} ${servo_width + 0.01} ${bracket_height/4}"/> -->
+        </geometry>
+        <material name="bracket_gray"/>
+      </visual>
+      <collision>
         <origin xyz="0 0 ${bracket_height/2}" rpy="0 0 0"/>
         <geometry>
-          <box size="${mount_thickness} ${servo_width + 0.01} ${bracket_height/4}"/>
-        </geometry>
-        <material name="bracket_gray"/>
-      </visual>
-      <collision>
+          <mesh filename="file://$(find image_sync_processor)/meshes/stls/PAN-TILT_ROTOR_V2_fixed.stl" scale="0.001 0.001 0.001" />
+          <!-- <box size="${mount_thickness} ${servo_width + 0.01} ${bracket_height/4}"/> -->
+        </geometry>
+      </collision>
+      <inertial>
         <origin xyz="0 0 ${bracket_height/2}" rpy="0 0 0"/>
-        <geometry>
-          <box size="${mount_thickness} ${servo_width + 0.01} ${bracket_height/4}"/>
-        </geometry>
-      </collision>
-      <inertial>
-        <origin xyz="0 0 ${bracket_height/4}" rpy="0 0 0"/>
         <mass value="0.02"/>
         <inertia ixx="0.000005" ixy="0.0" ixz="0.0"
@@ -143,5 +151,6 @@
     </link>
     <joint name="pan_joint" type="revolute">
-      <origin xyz="0 0 ${servo_height/2 + servo_horn_height}" rpy="0 0 0"/>
+      <!-- <origin xyz="0 0 ${servo_height/2 + servo_horn_height}" rpy="0 0 0"/> -->
+      <origin xyz="0 0 ${servo_height + servo_horn_height}" rpy="0 0 0"/>
       <parent link="pan_servo_link"/>
       <child link="pan_link"/>
@@ -177,5 +186,5 @@
     </link>
     <joint name="tilt_servo_joint" type="fixed">
-      <origin xyz="0 0 ${bracket_height-0.01}" rpy="0 0 0"/>
+      <origin xyz="0 0 ${mount_thickness*2}" rpy="0 0 0"/>
       <parent link="pan_link"/>
       <child link="tilt_servo_link"/>
@@ -221,7 +230,8 @@
     <link name="pan_tilt_camera_link">
       <visual>
-        <origin xyz="0 0 0" rpy="0 0 0"/>
-        <geometry>
-          <box size="${camera_length} ${camera_width} ${camera_height}"/>
+        <origin xyz="0 0 0" rpy="0 0 1.57"/>
+        <geometry>
+          <mesh filename="file://$(find image_sync_processor)/meshes/stls/pi_stand_final_v2-Body_v2_fixed.stl" scale="0.001 0.001 0.001" />
+          <!-- <box size="${camera_length} ${camera_width} ${camera_height}"/> -->
         </geometry>
         <material name="camera_black"/>
@@ -242,5 +252,5 @@
     </link>
     <joint name="camera_mount_joint" type="fixed">
-      <origin xyz="0 -${camera_height + servo_height} 0" rpy="0 1.57 -1.57"/>
+      <origin xyz="0 -${pan_tilt_leg_h/2 +0.022+ camera_mount_h/2} 0" rpy="0 1.57 -1.57"/>
       <!-- <origin xyz="0 0 0" rpy="0 0 0"/> -->
       <parent link="tilt_link"/>

File: ros_ws/src/autonomous_robot/description/pan_tilt_xacros/pan_tilt_test.xacro (robot description, xacro)
@@ -5,5 +5,5 @@
   <link name="base_link">
     <visual>
-      <origin xyz="0 0 0.05" rpy="0 0 0"/>
+      <origin xyz="0 0 0.005" rpy="0 0 0"/>
       <geometry>
         <box size="0.1 0.1 0.01"/>
@@ -14,5 +14,5 @@
     </visual>
     <collision>
-      <origin xyz="0 0 0.05" rpy="0 0 0"/>
+      <origin xyz="0 0 0.005" rpy="0 0 0"/>
       <geometry>
         <box size="0.1 0.1 0.01"/>
@@ -20,5 +20,5 @@
     </collision>
     <inertial>
-      <origin xyz="0 0 0.05" rpy="0 0 0"/>
+      <origin xyz="0 0 0.005" rpy="0 0 0"/>
       <mass value="0.1"/>
       <inertia ixx="0.0001" ixy="0.0" ixz="0.0"
@@ -29,5 +29,5 @@
   <!-- Instantiate the pan-tilt mechanism -->
   <xacro:pan_tilt_mechanism parent="base_link">
-    <origin xyz="0 0 0.1" rpy="0 0 0"/>
+    <origin xyz="0 0 0.01" rpy="0 0 0"/>
   </xacro:pan_tilt_mechanism>
 </robot>

Commit message: update camera pan tilt

File: ros_ws/src/autonomous_robot/description/pan_tilt_xacros/pan_tilt.xacro (robot description, xacro)
@@ -78,5 +78,6 @@
         <origin xyz="0 0 ${servo_height/2}" rpy="1.57 0 0"/>
         <geometry>
-          <mesh filename="file://$(find image_sync_processor)/meshes/stls/PAN-TILT_BASE_V1_fixed.dae" scale="0.001 0.001 0.001" />
+          <mesh filename="file://$(find image_sync_processor)/meshes/stls/PAN-TILT_BASE_V1_fixed.stl" scale="0.001 0.001 0.001" />
+          <!-- <mesh filename="file://$(find image_sync_processor)/meshes/stls/PAN-TILT_BASE_V1_fixed.dae" scale="0.001 0.001 0.001" /> -->
           <!-- <box size="${servo_length} ${servo_width} ${servo_height}"/> -->
         </geometry>
@@ -136,5 +137,6 @@
       </visual>
       <collision>
-        <origin xyz="0 0 ${bracket_height/2}" rpy="0 0 0"/>
+        <!-- <origin xyz="0 0 ${bracket_height/2}" rpy="0 0 0"/> -->
+        <origin xyz="0 0 0" rpy="0 0 0"/>
         <geometry>
           <mesh filename="file://$(find image_sync_processor)/meshes/stls/PAN-TILT_ROTOR_V2_fixed.stl" scale="0.001 0.001 0.001" />
@@ -143,5 +145,6 @@
       </collision>
       <inertial>
-        <origin xyz="0 0 ${bracket_height/2}" rpy="0 0 0"/>
+        <!-- <origin xyz="0 0 ${bracket_height/2}" rpy="0 0 0"/> -->
+        <origin xyz="0 0 0" rpy="0 0 0"/>
         <mass value="0.02"/>
         <inertia ixx="0.000005" ixy="0.0" ixz="0.0"
@@ -202,5 +205,5 @@
       </visual>
       <collision>
-        <origin xyz="0 0 0" rpy="0 0 0"/>
+        <origin xyz="0 -0.022 0" rpy="0 0 0"/>
         <!-- <origin xyz="-${servo_length/4 + 0.01} 0 ${servo_length}" rpy="-1.57 0 1.57"/> -->
         <geometry>
@@ -210,5 +213,5 @@
       </collision>
       <inertial>
-        <origin xyz="0 0 0" rpy="0 0 0"/>
+        <origin xyz="0 -0.022 0" rpy="0 0 0"/>
         <!-- <origin xyz="-${servo_length/4 + 0.01} 0 ${servo_length}" rpy="-1.57 0 1.57"/> -->
         <mass value="0.02"/>
@@ -238,11 +241,12 @@
       </visual>
       <collision>
-        <origin xyz="0 0 0" rpy="0 0 0"/>
-        <geometry>
-          <box size="${camera_length} ${camera_width} ${camera_height}"/>
-        </geometry>
-      </collision>
-      <inertial>
-        <origin xyz="0 0 0" rpy="0 0 0"/>
+        <origin xyz="0 0 0" rpy="0 0 1.57"/>
+        <geometry>
+          <!-- <box size="${camera_length} ${camera_width} ${camera_height}"/> -->
+          <mesh filename="file://$(find image_sync_processor)/meshes/stls/pi_stand_final_v2-Body_v2_fixed.stl" scale="0.001 0.001 0.001" />
+        </geometry>
+      </collision>
+      <inertial>
+        <origin xyz="0 0 0" rpy="0 0 1.57"/>
         <mass value="0.01"/>
         <inertia ixx="0.000001" ixy="0.0" ixz="0.0"

File: ros_ws/src/autonomous_robot/description/pan_tilt_xacros/robot_pan_tilt.xacro (robot description, xacro)
@@ -4,5 +4,5 @@
   <!-- Instantiate the pan-tilt mechanism -->
   <xacro:pan_tilt_mechanism parent="chassis">
-    <origin xyz="${chassis_length/2} -${chassis_width/4} ${chassis_height+0.1}" rpy="0 0.18 0"/>
+    <origin xyz="${chassis_length/2} -${chassis_width/4} ${chassis_height+0.01}" rpy="0 0.18 0"/>
   </xacro:pan_tilt_mechanism>
 </robot>

Commit message: update camera pan tilt

File: ros_ws/src/autonomous_robot/description/pan_tilt_xacros/pan_tilt.xacro (robot description, xacro)
@@ -80,5 +80,5 @@
           <mesh filename="file://$(find image_sync_processor)/meshes/stls/PAN-TILT_BASE_V1_fixed.stl" scale="0.001 0.001 0.001" />
           <!-- <mesh filename="file://$(find image_sync_processor)/meshes/stls/PAN-TILT_BASE_V1_fixed.dae" scale="0.001 0.001 0.001" /> -->
-          <!-- <box size="${servo_length} ${servo_width} ${servo_height}"/> -->
+          <!-- <box size="0.06 0.06 0.06"/> -->
         </geometry>
       </collision>
@@ -137,5 +137,4 @@
       </visual>
       <collision>
-        <!-- <origin xyz="0 0 ${bracket_height/2}" rpy="0 0 0"/> -->
         <origin xyz="0 0 0" rpy="0 0 0"/>
         <geometry>
@@ -145,5 +144,4 @@
       </collision>
       <inertial>
-        <!-- <origin xyz="0 0 ${bracket_height/2}" rpy="0 0 0"/> -->
         <origin xyz="0 0 0" rpy="0 0 0"/>
         <mass value="0.02"/>

File: ros_ws/src/autonomous_robot/description/robot.urdf.xacro (robot description, xacro)
@@ -12,4 +12,5 @@
     <xacro:include filename="lidar.xacro" />
     <xacro:include filename="pan_tilt_xacros/robot_pan_tilt.xacro" />
+    <xacro:include filename="pan_tilt_xacros/ros2_control_pan_tilt.xacro" />
     <!-- <xacro:include filename="camera.xacro" /> -->
     <xacro:include filename="xarm_xacros/xarm.xacro" />

Commit message: update camera pan tilt

File: ros_ws/src/autonomous_robot/description/pan_tilt_xacros/pan_tilt.xacro (robot description, xacro)
@@ -17,9 +17,9 @@
     <xacro:property name="camera_width" value="0.025"/>
     <xacro:property name="camera_height" value="0.025"/>
-    <xacro:property name="camera_mount_l" value="0.09"/>
-    <xacro:property name="camera_mount_w" value="0.068"/>
+    <xacro:property name="camera_mount_w" value="0.09"/>
+    <xacro:property name="camera_mount_l" value="0.068"/>
     <xacro:property name="camera_mount_h" value="0.085"/>
     <xacro:property name="pan_tilt_leg_l" value="0.025"/>
-    <xacro:property name="pan_tilt_leg_2" value="0.058"/>
+    <xacro:property name="pan_tilt_leg_w" value="0.058"/>
     <xacro:property name="pan_tilt_leg_h" value="0.065"/>
     <!-- Mount Properties -->
@@ -35,4 +35,10 @@
     <material name="camera_black">
       <color rgba="0.05 0.05 0.05 1.0"/>
+    </material>
+    <material name="camera_red">
+      <color rgba="0.8 0.05 0.05 1.0"/>
+    </material>
+    <material name="camera_blue">
+      <color rgba="0.05 0.05 0.8 1.0"/>
     </material>
     <!-- Base Link -->
@@ -236,5 +242,5 @@
           <!-- <box size="${camera_length} ${camera_width} ${camera_height}"/> -->
         </geometry>
-        <material name="camera_black"/>
+        <material name="camera_blue"/>
       </visual>
       <collision>
@@ -259,11 +265,63 @@
       <child link="pan_tilt_camera_link"/>
     </joint>
+    <!-- Camera Link -->
+    <link name="rgb_camera_link">
+      <visual>
+        <origin xyz="0 0 0" rpy="0 0 0"/>
+        <geometry>
+          <box size="${camera_length} ${camera_width} ${camera_height}"/>
+        </geometry>
+        <material name="camera_red"/>
+      </visual>
+      <collision>
+        <origin xyz="0 0 0" rpy="0 0 0"/>
+        <geometry>
+          <box size="${camera_length} ${camera_width} ${camera_height}"/>
+        </geometry>
+      </collision>
+      <inertial>
+        <origin xyz="0 0 0" rpy="0 0 0"/>
+        <mass value="0.01"/>
+        <inertia ixx="0.000001" ixy="0.0" ixz="0.0"
+                 iyy="0.000001" iyz="0.0"
+                 izz="0.000001"/>
+      </inertial>
+    </link>
+    <joint name="rgb_camera_joint" type="fixed">
+      <origin xyz="${camera_mount_l/2} 0 0" rpy="0 0 0"/>
+      <!-- <origin xyz="0 0 0" rpy="0 0 0"/> -->
+      <parent link="pan_tilt_camera_link"/>
+      <child link="rgb_camera_link"/>
+    </joint>
     <!-- Camera Optical Frame (for proper ROS camera convention) -->
-    <link name="pan_tilt_camera_optical_link"/>
+    <link name="rgb_camera_optical_link"/>
     <joint name="camera_optical_joint" type="fixed">
       <origin xyz="0 0 0" rpy="${-pi/2} 0 ${-pi/2}"/>
-      <parent link="pan_tilt_camera_link"/>
-      <child link="pan_tilt_camera_optical_link"/>
+      <parent link="rgb_camera_link"/>
+      <child link="rgb_camera_optical_link"/>
     </joint>
   </xacro:macro>
+  <gazebo reference="rgb_camera_link">
+    <material>Gazebo/Black</material>
+    <sensor name="camera" type="camera">
+      <pose> 0 0 0 0 0 0 </pose>
+      <visualize>true</visualize>
+      <update_rate>10</update_rate>
+      <camera>
+        <camera_info_topic>camera/camera_info</camera_info_topic>
+        <horizontal_fov>1.089</horizontal_fov>
+        <image>
+          <format>R8G8B8</format>
+          <width>640</width>
+          <height>480</height>
+        </image>
+        <clip>
+          <near>0.05</near>
+          <far>8.0</far>
+        </clip>
+      </camera>
+      <topic>camera/image_raw</topic>
+      <gz_frame_id>rgb_camera_optical_link</gz_frame_id>
+  </sensor>
+  </gazebo>
 </robot>

File: ros_ws/src/autonomous_robot/description/pan_tilt_xacros/robot_pan_tilt.xacro (robot description, xacro)
@@ -4,5 +4,5 @@
   <!-- Instantiate the pan-tilt mechanism -->
   <xacro:pan_tilt_mechanism parent="chassis">
-    <origin xyz="${chassis_length/2} -${chassis_width/4} ${chassis_height+0.01}" rpy="0 0.18 0"/>
+    <origin xyz="${chassis_length/2} -${chassis_width/4} ${chassis_height+0.005}" rpy="0 0.0 0"/>
   </xacro:pan_tilt_mechanism>
 </robot>

Commit message: pan tilt stuff

File: ros_ws/src/autonomous_robot/description/pan_tilt_xacros/pan_tilt.xacro (robot description, xacro)
@@ -14,7 +14,7 @@
     <xacro:property name="base_height" value="0.01"/>
     <!-- Camera Properties -->
-    <xacro:property name="camera_length" value="0.025"/>
-    <xacro:property name="camera_width" value="0.025"/>
-    <xacro:property name="camera_height" value="0.025"/>
+    <xacro:property name="camera_length" value="0.02"/>
+    <xacro:property name="camera_width" value="0.028"/>
+    <xacro:property name="camera_height" value="0.027"/>
     <xacro:property name="camera_mount_w" value="0.09"/>
     <xacro:property name="camera_mount_l" value="0.068"/>
@@ -159,5 +159,5 @@
     <joint name="pan_joint" type="revolute">
       <!-- <origin xyz="0 0 ${servo_height/2 + servo_horn_height}" rpy="0 0 0"/> -->
-      <origin xyz="0 0 ${servo_height + servo_horn_height}" rpy="0 0 0"/>
+      <origin xyz="-${servo_length/4} 0 ${servo_height + servo_horn_height}" rpy="0 0 0"/>
       <parent link="pan_servo_link"/>
       <child link="pan_link"/>
@@ -193,5 +193,5 @@
     </link>
     <joint name="tilt_servo_joint" type="fixed">
-      <origin xyz="0 0 ${mount_thickness*2}" rpy="0 0 0"/>
+      <origin xyz="0 ${servo_height/4} ${mount_thickness*2}" rpy="0 0 0"/>
       <parent link="pan_link"/>
       <child link="tilt_servo_link"/>
@@ -289,5 +289,5 @@
     </link>
     <joint name="rgb_camera_joint" type="fixed">
-      <origin xyz="${camera_mount_l/2} 0 0" rpy="0 0 0"/>
+      <origin xyz="${camera_mount_l/2} 0.024 -0.004" rpy="0 0 0"/>
       <!-- <origin xyz="0 0 0" rpy="0 0 0"/> -->
       <parent link="pan_tilt_camera_link"/>
