Commit message: updates

File: ros_ws/src/autonomous_robot/description/pan_tilt_xacros/pan_tilt_test.xacro (robot description, xacro)
@@ -1,5 +1,5 @@
 <?xml version="1.0"?>
 <robot name="pan_tilt_test" xmlns:xacro="http://www.ros.org/wiki/xacro">
-  <xacro:include filename="$(find autonomous_robot)/description/pan_tilt_xacros/pan_tilt.xacro"/>
+  <xacro:include filename="$(find autonomous_robot)/description/pan_tilt_xacros/pan_tilt_old.xacro"/>
   <!-- Base link -->
   <link name="base_link">

File: ros_ws/src/autonomous_robot/description/pan_tilt_xacros/robot_pan_tilt.xacro (robot description, xacro)
@@ -5,5 +5,6 @@
   <!-- Instantiate the pan-tilt mechanism -->
   <xacro:pan_tilt_mechanism parent="chassis">
-    <origin xyz="${chassis_length/2} -${chassis_width/4} ${chassis_height+0.005}" rpy="0 0.0 0"/>
+    <origin xyz="${chassis_length/2-0.08+0.028} -${chassis_width/2-0.088+0.04} ${chassis_height}" rpy="0 0.0 0"/>
   </xacro:pan_tilt_mechanism>
+  <xacro:include filename="$(find pan_tilt_description)/urdf/ros2_control_pan_tilt.xacro"/>
 </robot>

File: ros_ws/src/autonomous_robot/description/robot.urdf.xacro (robot description, xacro)
@@ -12,5 +12,4 @@
     <xacro:include filename="lidar.xacro" />
     <xacro:include filename="pan_tilt_xacros/robot_pan_tilt.xacro" />
-    <xacro:include filename="$(find pan_tilt_description)/urdf/ros2_control_pan_tilt.xacro"/>
     <!-- <xacro:include filename="pan_tilt_xacros/ros2_control_pan_tilt.xacro" /> -->
     <!-- <xacro:include filename="camera.xacro" /> -->

File: ros_ws/src/autonomous_robot/description/xarm_xacros/xarm.xacro (robot description, xacro)
@@ -14,5 +14,5 @@
         <parent link="chassis"/>
         <child link="xarm_base_link"/>
-        <origin xyz="${chassis_length1/4+0.02} ${chassis_width1/4+0.02} ${chassis_height1}" rpy="0.0 0.0 -${pi/2}"/>
+        <origin xyz="${chassis_length1/2-0.08} ${chassis_width1/2-0.08} ${chassis_height1}" rpy="0.0 0.0 -${pi/2}"/>
     </joint>
     <xacro:property name="sim_mode" value="true"/>

File: ros_ws/src/pan_tilt_description/urdf/pan_tilt.xacro (robot description, xacro)
@@ -227,5 +227,5 @@
     <joint name="tilt_joint" type="revolute">
       <!-- <origin xyz="0 0 0" rpy="0 0 0"/> -->
-      <origin xyz="${servo_length/2} 0 ${servo_height/10}" rpy="-1.57 0 1.57"/>
+      <origin xyz="${servo_length/2} 0.01 ${servo_height/10}" rpy="-1.57 0 1.57"/>
       <parent link="tilt_servo_link"/>
       <child link="tilt_link"/>
@@ -303,4 +303,74 @@
   </xacro:macro>
   <gazebo reference="rgb_camera_link">
+    <sensor name="depth_camera" type="depth_camera">
+      <camera>
+        <horizontal_fov>1.25</horizontal_fov>
+        <image>
+          <width>320</width>
+          <height>240</height>
+          <format>R8G8B8</format>
+          <!-- <format>L16</format> -->
+        </image>
+        <clip>
+          <near>0.1</near>
+          <far>20</far>
+        </clip>
+        <!-- <optical_frame_id>camera_link</optical_frame_id> -->
+        <optical_frame_id>rgb_camera_optical_link</optical_frame_id>
+        <camera_info_topic>camera/depth/camera_info</camera_info_topic>
+      </camera>
+      <always_on>1</always_on>
+      <update_rate>20</update_rate>
+      <visualize>true</visualize>
+      <topic>camera/depth/image_raw</topic>
+      <point_cloud_topic>camera/depth/points</point_cloud_topic>
+      <gz_frame_id>rgb_camera_link</gz_frame_id>
+    </sensor>
+    <sensor name="camera" type="camera">
+      <camera>
+        <horizontal_fov>1.25</horizontal_fov>
+        <image>
+          <width>320</width>
+          <height>240</height>
+          <format>R8G8B8</format>
+        </image>
+        <clip>
+          <near>0.1</near>
+          <far>20</far>
+        </clip>
+        <optical_frame_id>rgb_camera_optical_link</optical_frame_id>
+        <camera_info_topic>camera/camera_info</camera_info_topic>
+      </camera>
+      <always_on>1</always_on>
+      <update_rate>20</update_rate>
+      <visualize>true</visualize>
+      <topic>camera/image_raw</topic>
+      <!-- <gz_frame_id>rgb_camera_link</gz_frame_id> -->
+    </sensor>
+  </gazebo>
+  <!-- <gazebo reference="rgb_camera_link">
+    <material>Gazebo/Black</material>
+    <sensor name="camera" type="depth_camera">
+      <pose> 0 0 0 0 0 0 </pose>
+      <visualize>true</visualize>
+      <update_rate>10</update_rate>
+      <camera>
+        <camera_info_topic>camera/camera_info</camera_info_topic>
+        <horizontal_fov>1.089</horizontal_fov>
+        <image>
+          <format>R8G8B8</format>
+          <width>640</width>
+          <height>480</height>
+        </image>
+        <clip>
+          <near>0.05</near>
+          <far>8.0</far>
+        </clip>
+      </camera>
+      <topic>camera/image_raw</topic>
+      <gz_frame_id>rgb_camera_optical_link</gz_frame_id>
+    </sensor>
+  </gazebo> -->
+  <!-- <gazebo reference="rgb_camera_link">
     <material>Gazebo/Black</material>
     <sensor name="camera" type="camera">
@@ -324,4 +394,4 @@
       <gz_frame_id>rgb_camera_optical_link</gz_frame_id>
   </sensor>
-  </gazebo>
+  </gazebo> -->
 </robot>

Commit message: teleop pantilt

File: ros_ws/src/autonomous_robot/description/pan_tilt_xacros/pan_tilt_test.xacro (robot description, xacro)
@@ -1,5 +1,5 @@
 <?xml version="1.0"?>
 <robot name="pan_tilt_test" xmlns:xacro="http://www.ros.org/wiki/xacro">
-  <xacro:include filename="$(find autonomous_robot)/description/pan_tilt_xacros/pan_tilt_old.xacro"/>
+  <xacro:include filename="$(find pan_tilt_description)/urdf/pan_tilt.xacro"/>
   <!-- Base link -->
   <link name="base_link">

File: ros_ws/src/pan_tilt_description/urdf/pan_tilt.xacro (robot description, xacro)
@@ -227,5 +227,5 @@
     <joint name="tilt_joint" type="revolute">
       <!-- <origin xyz="0 0 0" rpy="0 0 0"/> -->
-      <origin xyz="${servo_length/2} 0.01 ${servo_height/10}" rpy="-1.57 0 1.57"/>
+      <origin xyz="${servo_length/2} 0.01 ${servo_height/10}" rpy="-1.4 0 1.57"/>
       <parent link="tilt_servo_link"/>
       <child link="tilt_link"/>
