Commit message: moved stls

File: ros_ws/src/pan_tilt_description/urdf/pan_tilt.xacro (robot description, xacro)
@@ -76,5 +76,5 @@
         <geometry>
           <!-- <mesh filename="file://$(find xarm_description)/meshes/stls/link5.stl" scale="1.0 1.0 1.0" /> -->
-          <mesh filename="file://$(find image_sync_processor)/meshes/stls/PAN-TILT_BASE_V1_fixed.stl" scale="0.001 0.001 0.001" />
+          <mesh filename="file://$(find pan_tilt_description)/urdf/meshes/stls/PAN-TILT_BASE_V1_fixed.stl" scale="0.001 0.001 0.001" />
           <!-- <box size="${servo_length} ${servo_width} ${servo_height}"/> -->
         </geometry>
@@ -84,6 +84,6 @@
         <origin xyz="0 0 ${servo_height/2}" rpy="1.57 0 0"/>
         <geometry>
-          <mesh filename="file://$(find image_sync_processor)/meshes/stls/PAN-TILT_BASE_V1_fixed.stl" scale="0.001 0.001 0.001" />
-          <!-- <mesh filename="file://$(find image_sync_processor)/meshes/stls/PAN-TILT_BASE_V1_fixed.dae" scale="0.001 0.001 0.001" /> -->
+          <mesh filename="file://$(find pan_tilt_description)/urdf/meshes/stls/PAN-TILT_BASE_V1_fixed.stl" scale="0.001 0.001 0.001" />
+          <!-- <mesh filename="file://$(find pan_tilt_description)/urdf/meshes/stls/PAN-TILT_BASE_V1_fixed.dae" scale="0.001 0.001 0.001" /> -->
           <!-- <box size="0.06 0.06 0.06"/> -->
         </geometry>
@@ -107,5 +107,5 @@
         <geometry>
           <!-- <mesh filename="file://$(find xarm_description)/meshes/stls/link5.stl" scale="1.0 1.0 1.0" /> -->
-          <!-- <mesh filename="file://$(find image_sync_processor)/meshes/stls/PAN-TILT_BASE_V1_fixed.stl" scale="0.001 0.001 0.001" /> -->
+          <!-- <mesh filename="file://$(find pan_tilt_description)/urdf/meshes/stls/PAN-TILT_BASE_V1_fixed.stl" scale="0.001 0.001 0.001" /> -->
           <box size="${servo_length} ${servo_width} ${servo_height}"/>
         </geometry>
@@ -115,5 +115,5 @@
         <origin xyz="0 0 ${servo_height/2}" rpy="0 0 0"/>
         <geometry>
-          <!-- <mesh filename="file://$(find image_sync_processor)/meshes/stls/PAN-TILT_BASE_V1_fixed.dae" scale="0.001 0.001 0.001" /> -->
+          <!-- <mesh filename="file://$(find pan_tilt_description)/urdf/meshes/stls/PAN-TILT_BASE_V1_fixed.dae" scale="0.001 0.001 0.001" /> -->
           <box size="${servo_length} ${servo_width} ${servo_height}"/>
         </geometry>
@@ -137,5 +137,5 @@
         <origin xyz="0 0 0" rpy="0 0 0"/>
         <geometry>
-          <mesh filename="file://$(find image_sync_processor)/meshes/stls/PAN-TILT_ROTOR_V2_fixed.stl" scale="0.001 0.001 0.001" />
+          <mesh filename="file://$(find pan_tilt_description)/urdf/meshes/stls/PAN-TILT_ROTOR_V2_fixed.stl" scale="0.001 0.001 0.001" />
           <!-- <box size="${mount_thickness} ${servo_width + 0.01} ${bracket_height/4}"/> -->
         </geometry>
@@ -145,5 +145,5 @@
         <origin xyz="0 0 0" rpy="0 0 0"/>
         <geometry>
-          <mesh filename="file://$(find image_sync_processor)/meshes/stls/PAN-TILT_ROTOR_V2_fixed.stl" scale="0.001 0.001 0.001" />
+          <mesh filename="file://$(find pan_tilt_description)/urdf/meshes/stls/PAN-TILT_ROTOR_V2_fixed.stl" scale="0.001 0.001 0.001" />
           <!-- <box size="${mount_thickness} ${servo_width + 0.01} ${bracket_height/4}"/> -->
         </geometry>
@@ -204,5 +204,5 @@
         <geometry>
           <!-- <box size="${servo_length + 0.02} ${servo_width + 0.01} ${mount_thickness}"/> -->
-          <mesh filename="file://$(find image_sync_processor)/meshes/stls/PAN-TILT_LEG_V2_fixed.stl" scale="0.001 0.001 0.001" />
+          <mesh filename="file://$(find pan_tilt_description)/urdf/meshes/stls/PAN-TILT_LEG_V2_fixed.stl" scale="0.001 0.001 0.001" />
         </geometry>
         <material name="bracket_gray"/>
@@ -213,5 +213,5 @@
         <geometry>
           <!-- <box size="${servo_length + 0.02} ${servo_width + 0.01} ${mount_thickness}"/> -->
-          <mesh filename="file://$(find image_sync_processor)/meshes/stls/PAN-TILT_LEG_V2_fixed.stl" scale="0.001 0.001 0.001" />
+          <mesh filename="file://$(find pan_tilt_description)/urdf/meshes/stls/PAN-TILT_LEG_V2_fixed.stl" scale="0.001 0.001 0.001" />
         </geometry>
       </collision>
@@ -239,5 +239,5 @@
         <origin xyz="0 0 0" rpy="0 0 1.57"/>
         <geometry>
-          <mesh filename="file://$(find image_sync_processor)/meshes/stls/pi_stand_final_v2-Body_v2_fixed.stl" scale="0.001 0.001 0.001" />
+          <mesh filename="file://$(find pan_tilt_description)/urdf/meshes/stls/pi_stand_final_v2-Body_v2_fixed.stl" scale="0.001 0.001 0.001" />
           <!-- <box size="${camera_length} ${camera_width} ${camera_height}"/> -->
         </geometry>
@@ -248,5 +248,5 @@
         <geometry>
           <!-- <box size="${camera_length} ${camera_width} ${camera_height}"/> -->
-          <mesh filename="file://$(find image_sync_processor)/meshes/stls/pi_stand_final_v2-Body_v2_fixed.stl" scale="0.001 0.001 0.001" />
+          <mesh filename="file://$(find pan_tilt_description)/urdf/meshes/stls/pi_stand_final_v2-Body_v2_fixed.stl" scale="0.001 0.001 0.001" />
         </geometry>
       </collision>

Commit message: updated pan tilt

File: ros_ws/src/pan_tilt_description/urdf/pan_tilt.xacro (robot description, xacro)
@@ -200,5 +200,5 @@
     <link name="tilt_link">
       <visual>
-        <origin xyz="0 -0.022 0" rpy="0 0 0"/>
+        <origin xyz="0 -0.0022 0" rpy="0 0 0"/>
         <!-- <origin xyz="-${servo_length/4 + 0.01} 0 ${servo_length}" rpy="-1.57 0 1.57"/> -->
         <geometry>
@@ -209,5 +209,5 @@
       </visual>
       <collision>
-        <origin xyz="0 -0.022 0" rpy="0 0 0"/>
+        <origin xyz="0 -0.0022 0" rpy="0 0 0"/>
         <!-- <origin xyz="-${servo_length/4 + 0.01} 0 ${servo_length}" rpy="-1.57 0 1.57"/> -->
         <geometry>
@@ -217,5 +217,5 @@
       </collision>
       <inertial>
-        <origin xyz="0 -0.022 0" rpy="0 0 0"/>
+        <origin xyz="0 -0.0022 0" rpy="0 0 0"/>
         <!-- <origin xyz="-${servo_length/4 + 0.01} 0 ${servo_length}" rpy="-1.57 0 1.57"/> -->
         <mass value="0.02"/>
@@ -260,5 +260,5 @@
     </link>
     <joint name="camera_mount_joint" type="fixed">
-      <origin xyz="0 -${pan_tilt_leg_h/2 +0.022+ camera_mount_h/2} 0" rpy="0 1.57 -1.57"/>
+      <origin xyz="0 -${pan_tilt_leg_h/2 +0.002+ camera_mount_h/2} 0" rpy="0 1.57 -1.57"/>
       <!-- <origin xyz="0 0 0" rpy="0 0 0"/> -->
       <parent link="tilt_link"/>

Commit message: updated pan tilt

File: ros_ws/src/pan_tilt_description/urdf/pan_tilt.xacro (robot description, xacro)
@@ -260,5 +260,5 @@
     </link>
     <joint name="camera_mount_joint" type="fixed">
-      <origin xyz="0 -${pan_tilt_leg_h/2 +0.002+ camera_mount_h/2} 0" rpy="0 1.57 -1.57"/>
+      <origin xyz="0 -${pan_tilt_leg_h/2 +0.022+ camera_mount_h/2} 0" rpy="0 1.57 -1.57"/>
       <!-- <origin xyz="0 0 0" rpy="0 0 0"/> -->
       <parent link="tilt_link"/>

Commit message: updated pan tilt

File: ros_ws/src/pan_tilt_description/urdf/pan_tilt.xacro (robot description, xacro)
@@ -200,5 +200,5 @@
     <link name="tilt_link">
       <visual>
-        <origin xyz="0 -0.0022 0" rpy="0 0 0"/>
+        <origin xyz="0 -0.022 0" rpy="0 0 0"/>
         <!-- <origin xyz="-${servo_length/4 + 0.01} 0 ${servo_length}" rpy="-1.57 0 1.57"/> -->
         <geometry>
@@ -209,5 +209,5 @@
       </visual>
       <collision>
-        <origin xyz="0 -0.0022 0" rpy="0 0 0"/>
+        <origin xyz="0 -0.022 0" rpy="0 0 0"/>
         <!-- <origin xyz="-${servo_length/4 + 0.01} 0 ${servo_length}" rpy="-1.57 0 1.57"/> -->
         <geometry>
@@ -217,5 +217,5 @@
       </collision>
       <inertial>
-        <origin xyz="0 -0.0022 0" rpy="0 0 0"/>
+        <origin xyz="0 -0.022 0" rpy="0 0 0"/>
         <!-- <origin xyz="-${servo_length/4 + 0.01} 0 ${servo_length}" rpy="-1.57 0 1.57"/> -->
         <mass value="0.02"/>

Commit message: updated pan tilt

File: ros_ws/src/pan_tilt_description/urdf/pan_tilt.xacro (robot description, xacro)
@@ -227,5 +227,5 @@
     <joint name="tilt_joint" type="revolute">
       <!-- <origin xyz="0 0 0" rpy="0 0 0"/> -->
-      <origin xyz="${servo_length/2} 0.01 ${servo_height/10}" rpy="-1.4 0 1.57"/>
+      <origin xyz="${servo_length/2-0.01} 0.005 ${servo_height/10}" rpy="-1.4 0 1.57"/>
       <parent link="tilt_servo_link"/>
       <child link="tilt_link"/>

Commit message: updated pan tilt

File: ros_ws/src/pan_tilt_description/urdf/pan_tilt.xacro (robot description, xacro)
@@ -200,5 +200,5 @@
     <link name="tilt_link">
       <visual>
-        <origin xyz="0 -0.022 0" rpy="0 0 0"/>
+        <origin xyz="0 -0.0022 0" rpy="0 0 0"/>
         <!-- <origin xyz="-${servo_length/4 + 0.01} 0 ${servo_length}" rpy="-1.57 0 1.57"/> -->
         <geometry>
@@ -209,5 +209,5 @@
       </visual>
       <collision>
-        <origin xyz="0 -0.022 0" rpy="0 0 0"/>
+        <origin xyz="0 -0.0022 0" rpy="0 0 0"/>
         <!-- <origin xyz="-${servo_length/4 + 0.01} 0 ${servo_length}" rpy="-1.57 0 1.57"/> -->
         <geometry>
@@ -217,5 +217,5 @@
       </collision>
       <inertial>
-        <origin xyz="0 -0.022 0" rpy="0 0 0"/>
+        <origin xyz="0 -0.0022 0" rpy="0 0 0"/>
         <!-- <origin xyz="-${servo_length/4 + 0.01} 0 ${servo_length}" rpy="-1.57 0 1.57"/> -->
         <mass value="0.02"/>
@@ -227,5 +227,5 @@
     <joint name="tilt_joint" type="revolute">
       <!-- <origin xyz="0 0 0" rpy="0 0 0"/> -->
-      <origin xyz="${servo_length/2-0.01} 0.005 ${servo_height/10}" rpy="-1.4 0 1.57"/>
+      <origin xyz="${servo_length/2} 0.01 ${servo_height/10}" rpy="-1.4 0 1.57"/>
       <parent link="tilt_servo_link"/>
       <child link="tilt_link"/>
