Commit message: pan tilt stand alone

File: ros_ws/src/pan_tilt_hardware/urdf/pan_tilt_pi.urdf.xacro (robot description, xacro)
@@ -12,5 +12,5 @@
     <xacro:property name="base_length" value="0.06"/>
     <xacro:property name="base_width" value="0.06"/>
-    <xacro:property name="base_height" value="0.01"/>
+    <xacro:property name="base_height" value="0.025"/>
     <!-- Camera Properties -->
     <xacro:property name="camera_length" value="0.02"/>
@@ -216,5 +216,5 @@
     <joint name="tilt_joint" type="revolute">
       <!-- <origin xyz="0 0 0" rpy="0 0 0"/> -->
-      <origin xyz="${servo_length/2} 0.01 ${servo_height/10}" rpy="-1.57 0 1.57"/>
+      <origin xyz="${servo_length/2} 0.01 ${servo_height/10}" rpy="-1.4 0 1.57"/>
       <parent link="tilt_servo_link"/>
       <child link="tilt_link"/>

File: ros_ws/src/pan_tilt_hardware/urdf/pan_tilt_standalone_pi.xacro (robot description, xacro)
@@ -2,4 +2,8 @@
 <robot xmlns:xacro="http://www.ros.org/wiki/xacro" name="pan_tilt_robot">
   <xacro:arg name="sim_mode" default="false"/>
+  <!-- Include pan_tilt mechanism -->
+  <!-- <xacro:include filename="$(find pan_tilt_description)/urdf/pan_tilt.xacro"/> -->
+  <!-- Include ros2_control configuration -->
+  <!-- <xacro:include filename="$(find pan_tilt_description)/urdf/ros2_control_pan_tilt.xacro"/> -->
   <!-- Include pan_tilt mechanism -->
   <xacro:include filename="pan_tilt_pi.urdf.xacro"/>
