Commit message: cleanup

File: ros_ws/src/autonomous_robot/description/xarm_xacros/xarm.xacro (robot description, xacro)
@@ -16,5 +16,7 @@
         <origin xyz="${chassis_length1/4+0.02} ${chassis_width1/4+0.02} ${chassis_height1}" rpy="0.0 0.0 -${pi/2}"/>
     </joint>
+    <xacro:property name="sim_mode" value="true"/>
     <!-- <xacro:include filename="ros2_control.arm.xacro" /> -->
+    <!-- <xacro:include filename="ros2_control.arm copy.xacro" /> -->
     <xacro:include filename="$(find xarm_description)/urdf/ros2_control.arm.xacro"/>
 </robot>

File: ros_ws/src/xarm_description/urdf/ros2_control.arm.xacro (robot description, xacro)
@@ -111,5 +111,5 @@
   </xacro:unless>
   <xacro:if value="$(arg sim_mode)">
-    <ros2_control name="GazeboSystem" type="system">
+    <ros2_control name="arm_system" type="system">
         <hardware>
             <plugin>gz_ros2_control/GazeboSimSystem</plugin>

Commit message: got launch to work

File: ros_ws/src/autonomous_robot/description/xarm_xacros/xarm.xacro (robot description, xacro)
@@ -16,5 +16,4 @@
         <origin xyz="${chassis_length1/2-0.08} ${chassis_width1/2-0.08} ${chassis_height1}" rpy="0.0 0.0 -${pi/2}"/>
     </joint>
-    <xacro:property name="sim_mode" value="true"/>
     <!-- <xacro:include filename="ros2_control.arm.xacro" /> -->
     <!-- <xacro:include filename="ros2_control.arm copy.xacro" /> -->

Commit message: update robot arm

File: ros_ws/src/autonomous_robot/description/xarm_xacros/xarm.xacro (robot description, xacro)
@@ -14,5 +14,5 @@
         <parent link="chassis"/>
         <child link="xarm_base_link"/>
-        <origin xyz="${chassis_length1/2-0.08} ${chassis_width1/2-0.08} ${chassis_height1}" rpy="0.0 0.0 -${pi/2}"/>
+        <origin xyz="${chassis_length1/2-0.09} ${chassis_width1/2-0.08} ${chassis_height1}" rpy="0.0 0.0 -${pi/2}"/>
     </joint>
     <!-- <xacro:include filename="ros2_control.arm.xacro" /> -->

Commit message: updated pan tilt

File: ros_ws/src/autonomous_robot/description/xarm_xacros/xarm.xacro (robot description, xacro)
@@ -14,5 +14,5 @@
         <parent link="chassis"/>
         <child link="xarm_base_link"/>
-        <origin xyz="${chassis_length1/2-0.09} ${chassis_width1/2-0.08} ${chassis_height1}" rpy="0.0 0.0 -${pi/2}"/>
+        <origin xyz="${chassis_length1/2-0.07} ${chassis_width1/2-0.08} ${chassis_height1}" rpy="0.0 0.0 -${pi/2}"/>
     </joint>
     <!-- <xacro:include filename="ros2_control.arm.xacro" /> -->

File: ros_ws/src/pan_tilt_description/urdf/pan_tilt.xacro (robot description, xacro)
@@ -12,5 +12,5 @@
     <xacro:property name="base_length" value="0.06"/>
     <xacro:property name="base_width" value="0.06"/>
-    <xacro:property name="base_height" value="0.01"/>
+    <xacro:property name="base_height" value="0.025"/>
     <!-- Camera Properties -->
     <xacro:property name="camera_length" value="0.02"/>
@@ -227,5 +227,5 @@
     <joint name="tilt_joint" type="revolute">
       <!-- <origin xyz="0 0 0" rpy="0 0 0"/> -->
-      <origin xyz="${servo_length/2} 0.01 ${servo_height/10}" rpy="-1.4 0 1.57"/>
+      <origin xyz="${servo_length/4} 0.005 ${servo_height/10}" rpy="-1.4 0 1.57"/>
       <parent link="tilt_servo_link"/>
       <child link="tilt_link"/>

Commit message: updated angle for xarm 5

File: ros_ws/src/autonomous_robot/description/xarm_xacros/xarm.xacro (robot description, xacro)
@@ -14,5 +14,5 @@
         <parent link="chassis"/>
         <child link="xarm_base_link"/>
-        <origin xyz="${chassis_length1/2-0.07} ${chassis_width1/2-0.08} ${chassis_height1}" rpy="0.0 0.0 -${pi/2}"/>
+        <origin xyz="${chassis_length1/2-0.09} ${chassis_width1/2-0.08} ${chassis_height1}" rpy="0.0 0.0 -${pi/2}"/>
     </joint>
     <!-- <xacro:include filename="ros2_control.arm.xacro" /> -->

File: ros_ws/src/xarm_description/urdf/xarm_v2.urdf (robot description, URDF)
Before this commit: robot xarm, 9 links, 8 joints
Joints:
- joint finger_pinch_joint: origin xyz=0 0 0.11 rpy=0 0 0 -> xyz=0 0 0.13 rpy=0 0 0
- joint xarm_5_joint: origin xyz=0 -0.0022 0.03195 rpy=0 0 0 -> xyz=0 -0.0022 0.03195 rpy=-0.08 0 0
